Commit message: update
refactor names

File: urdf/5DoF-arm-kenny.urdf (robot description, URDF)
Before this commit: robot Brazo Robotico.SLDASM, 5 links, 4 joints
Links:
- link  link1: mass 0.019155 -> 0.0191547172964518; geometry collision mesh filename=package://5DoF-arm-kenny/meshes/ link1.STL; visual mesh filename=package://5DoF-arm-kenny/meshes/ link1.STL
- link base_link: mass 0.043248 -> 0.0432483576430209; geometry collision mesh filename=package://5DoF-arm-kenny/meshes/base_link.STL; visual mesh filename=package://5DoF-arm-kenny/meshes/base_link.STL
- link link 4: mass 0.0057062 -> 0.0057062055751799; geometry collision mesh filename=package://5DoF-arm-kenny/meshes/link 4.STL; visual mesh filename=package://5DoF-arm-kenny/meshes/link 4.STL
- link link2: mass 0.024964 -> 0.0249636399428571; geometry collision mesh filename=package://5DoF-arm-kenny/meshes/link2.STL; visual mesh filename=package://5DoF-arm-kenny/meshes/link2.STL
- link link3: mass 0.029564 -> 0.0295644975322909; geometry collision mesh filename=package://5DoF-arm-kenny/meshes/link3.STL; visual mesh filename=package://5DoF-arm-kenny/meshes/link3.STL

Commit message: x
x

File: urdf/5DoF-arm-kenny.urdf (robot description, URDF)
Before this commit: robot 5DoF-arm-kenny, 5 links, 4 joints
Links:
- removed link  link1
- removed link link 4
- removed link link2
- removed link link3
- added link L1, mass 0.024964; collision mesh filename=package://5DoF-arm-kenny/meshes/L1.STL; visual mesh filename=package://5DoF-arm-kenny/meshes/L1.STL
- added link L2, mass 0.10579; collision mesh filename=package://5DoF-arm-kenny/meshes/L2.STL; visual mesh filename=package://5DoF-arm-kenny/meshes/L2.STL
- added link L3, mass 0.0057062; collision mesh filename=package://5DoF-arm-kenny/meshes/L3.STL; visual mesh filename=package://5DoF-arm-kenny/meshes/L3.STL
- link base_link: mass 0.0432483576430209 -> 0.11287
Joints:
- removed joint j1
- removed joint j2
- removed joint j3
- removed joint primera rotacion
- added joint J1: type revolute, parent base_link, child L1, origin xyz=0.083264 0.11027 0.31677 rpy=2.1235E-17 0.51698 -1.877, axis 0.95347 -0.30148 0, limit effort=0 velocity=0
- added joint J2: type revolute, parent L1, child L2, origin xyz=0.13567 -0.01585 0.064748 rpy=-3.1416 0.51184 -3.1416, axis 0 1 0, limit effort=0 velocity=0
- added joint J3: type revolute, parent L2, child L3, origin xyz=0.01 0 -0.01 rpy=-1.3697E-17 0.072098 2.6158E-15, axis 0 1 0, limit effort=0 velocity=0
